Commit message: 312

File: src/articubot_one/description/depth_camera.xacro (robot description, xacro)
@@ -2,5 +2,5 @@
 <robot xmlns:xacro="http://www.ros.org/wiki/xacro" >
     <joint name="camera_joint" type="fixed">
-        <parent link="chassis"/>
+        <parent link="claw_support"/>
         <child link="camera_link"/>
         <origin xyz="0.315 0 0.07" rpy="0 0.18 0"/>

File: src/articubot_one/description/robot.urdf.xacro (robot description, xacro)
@@ -14,5 +14,5 @@
     <!-- <xacro:include filename="camera.xacro" /> -->
     <xacro:include filename="arm_robot.xacro" />
-    <!-- <xacro:include filename="depth_camera.xacro" /> -->
+    <xacro:include filename="depth_camera.xacro" />
     <xacro:include filename="face.xacro" />
 </robot>

Commit message: 21

File: src/articubot_one/description/depth_camera.xacro (robot description, xacro)
@@ -4,5 +4,5 @@
         <parent link="claw_support"/>
         <child link="camera_link"/>
-        <origin xyz="0.315 0 0.07" rpy="0 0.18 0"/>
+        <origin xyz="0.05 0 0.05" rpy="0 1.57 0"/>
     </joint>
     <link name="camera_link">

Commit message: 3

File: src/articubot_one/description/depth_camera.xacro (robot description, xacro)
@@ -4,5 +4,5 @@
         <parent link="claw_support"/>
         <child link="camera_link"/>
-        <origin xyz="0.05 0 0.05" rpy="0 1.57 0"/>
+        <origin xyz="-0.05 0 -0.05" rpy="0 1.57 0"/>
     </joint>
     <link name="camera_link">

Commit message: 3

File: src/articubot_one/description/depth_camera.xacro (robot description, xacro)
@@ -2,5 +2,5 @@
 <robot xmlns:xacro="http://www.ros.org/wiki/xacro" >
     <joint name="camera_joint" type="fixed">
-        <parent link="claw_support"/>
+        <parent link="arm_base_link"/>
         <child link="camera_link"/>
         <origin xyz="-0.05 0 -0.05" rpy="0 1.57 0"/>

Commit message: 13

File: src/articubot_one/description/depth_camera.xacro (robot description, xacro)
@@ -2,5 +2,5 @@
 <robot xmlns:xacro="http://www.ros.org/wiki/xacro" >
     <joint name="camera_joint" type="fixed">
-        <parent link="arm_base_link"/>
+        <parent link="claw_support"/>
         <child link="camera_link"/>
         <origin xyz="-0.05 0 -0.05" rpy="0 1.57 0"/>

Commit message: ew

File: src/articubot_one/description/depth_camera.xacro (robot description, xacro)
@@ -13,4 +13,10 @@
             <material name="red"/>
         </visual>
+        <collision>
+            <geometry>
+                <box size="0.010 0.03 0.03"/>
+            </geometry>
+            <material name="red"/>
+        </collision>
     </link>
     <joint name="camera_optical_joint" type="fixed">

File: src/articubot_one/description/robot.urdf.xacro (robot description, xacro)
@@ -15,4 +15,4 @@
     <xacro:include filename="arm_robot.xacro" />
     <xacro:include filename="depth_camera.xacro" />
-    <xacro:include filename="face.xacro" />
+    <!-- <xacro:include filename="face.xacro" /> -->
 </robot>
