Commit message: fix error

File: src/articubot_one/description/ros2_control.xacro (robot description, xacro)
@@ -3,5 +3,5 @@
     <xacro:property name="PI" value="3.14159265359" />
     <xacro:unless value="$(arg sim_mode)">
-        <ros2_control name="RealRobot" type="system">
+        <ros2_control name="articubot" type="system">
             <hardware>
                 <plugin>diffdrive_arduino/DiffDriveArduinoHardware</plugin>
@@ -36,8 +36,4 @@
                 </command_interface>
                 <state_interface name="position"/>
-                <state_interface name="velocity"/>
-                <state_interface name="effort"/>
-                <state_interface name="voltage"/>
-                <state_interface name="temperature"/>
             </joint>
             <joint name="forearm_hand_1_joint">
@@ -47,8 +43,4 @@
                 </command_interface>
                 <state_interface name="position"/>
-                <state_interface name="velocity"/>
-                <state_interface name="effort"/>
-                <state_interface name="voltage"/>
-                <state_interface name="temperature"/>
             </joint>
             <joint name="forearm_hand_2_joint">
@@ -58,8 +50,4 @@
                 </command_interface>
                 <state_interface name="position"/>
-                <state_interface name="velocity"/>
-                <state_interface name="effort"/>
-                <state_interface name="voltage"/>
-                <state_interface name="temperature"/>
             </joint>
             <joint name="forearm_hand_3_joint">
@@ -69,8 +57,4 @@
                 </command_interface>
                 <state_interface name="position"/>
-                <state_interface name="velocity"/>
-                <state_interface name="effort"/>
-                <state_interface name="voltage"/>
-                <state_interface name="temperature"/>
             </joint>
              <joint name="forearm_claw_joint">
@@ -80,8 +64,4 @@
                 </command_interface>
                 <state_interface name="position"/>
-                <state_interface name="velocity"/>
-                <state_interface name="effort"/>
-                <state_interface name="voltage"/>
-                <state_interface name="temperature"/>
             </joint>
             <joint name="joint_4">
@@ -91,20 +71,5 @@
                 </command_interface>
                 <state_interface name="position"/>
-                <state_interface name="velocity"/>
-                <state_interface name="effort"/>
-                <state_interface name="voltage"/>
-                <state_interface name="temperature"/>
             </joint>
-            <!-- <joint name="joint_5">
-                <command_interface name="position">
-                <param name="min">-${PI / 2}</param>
-                <param name="max">0.0</param>
-                </command_interface>
-                <state_interface name="position"/>
-                <state_interface name="velocity"/>
-                <state_interface name="effort"/>
-                <state_interface name="voltage"/>
-                <state_interface name="temperature"/>
-            </joint>  -->
             <joint name="joint_5">
                 <param name="mimic">joint_4</param>

Commit message: gd

File: src/articubot_one/description/ros2_control.xacro (robot description, xacro)
@@ -157,12 +157,12 @@
                 <state_interface name="effort"/> -->
             </joint>
-            <joint name="joint_5">
+            <!-- <joint name="joint_5">
                 <param name="mimic">joint_4</param>
                 <param name="multiplier">-1</param>
-                <!-- <command_interface name="position">
+                <command_interface name="position">
                 <param name="min">0.0</param>
                 <param name="max">${PI / 2}</param>
-                </command_interface> -->
-            </joint>
+                </command_interface>
+            </joint> -->
         </ros2_control>
     </xacro:if>

Commit message: d

File: src/articubot_one/description/ros2_control.xacro (robot description, xacro)
@@ -157,5 +157,5 @@
                 <state_interface name="effort"/> -->
             </joint>
-            <!-- <joint name="joint_5">
+            <joint name="joint_5">
                 <param name="mimic">joint_4</param>
                 <param name="multiplier">-1</param>
@@ -164,5 +164,5 @@
                 <param name="max">${PI / 2}</param>
                 </command_interface>
-            </joint> -->
+            </joint>
         </ros2_control>
     </xacro:if>

Commit message: dasd

File: src/articubot_one/description/ros2_control.xacro (robot description, xacro)
@@ -157,13 +157,13 @@
                 <state_interface name="effort"/> -->
             </joint>
-            <joint name="joint_5">
+            <!-- <joint name="joint_5">
                 <param name="mimic">joint_4</param>
                 <param name="multiplier">-1</param>
-                <!-- <command_interface name="position">
+                <command_interface name="position">
                 <param name="min">0.0</param>
                 <param name="max">${PI / 2}</param>
                 </command_interface>
-                <state_interface name="position"/> -->
-            </joint>
+                <state_interface name="position"/>
+            </joint> -->
         </ros2_control>
     </xacro:if>

Commit message: test

File: src/articubot_one/description/ros2_control.xacro (robot description, xacro)
@@ -72,5 +72,5 @@
                 <state_interface name="position"/>
             </joint>
-            <joint name="joint_5">
+            <!-- <joint name="joint_5">
                 <param name="mimic">joint_4</param>
                 <param name="multiplier">-1</param>
@@ -79,5 +79,5 @@
                 <param name="max">${PI / 2}</param>
                 </command_interface>
-            </joint>
+            </joint> -->
         </ros2_control>
     </xacro:unless>

Commit message: 545

File: src/articubot_one/description/ros2_control.xacro (robot description, xacro)
@@ -72,5 +72,5 @@
                 <state_interface name="position"/>
             </joint>
-            <!-- <joint name="joint_5">
+            <joint name="joint_5">
                 <param name="mimic">joint_4</param>
                 <param name="multiplier">-1</param>
@@ -79,5 +79,5 @@
                 <param name="max">${PI / 2}</param>
                 </command_interface>
-            </joint> -->
+            </joint>
         </ros2_control>
     </xacro:unless>

Commit message: wq

File: src/articubot_one/description/ros2_control.xacro (robot description, xacro)
@@ -1,5 +1,5 @@
 <?xml version="1.0"?>
 <robot xmlns:xacro="http://www.ros.org/wiki/xacro">
-    <xacro:property name="pi" value="3.14159265359" />
+    <xacro:property name="PI" value="3.14159265359" />
     <xacro:unless value="$(arg sim_mode)">
         <ros2_control name="articubot" type="system">
@@ -35,6 +35,6 @@
             <joint name="arm_base_forearm_joint">
                 <command_interface name="position">
-                <param name="min">-${2*pi/3}</param>
-                <param name="max">${2*pi/3}</param>
+                <param name="min">-${2*PI/3}</param>
+                <param name="max">${2*PI/3}</param>
                 </command_interface>
                 <state_interface name="position"/>
@@ -42,6 +42,6 @@
             <joint name="forearm_hand_1_joint">
                 <command_interface name="position">
-                <param name="min">-${2*pi/3}</param>
-                <param name="max">${2*pi/3}</param>
+                <param name="min">-${2*PI/3}</param>
+                <param name="max">${2*PI/3}</param>
                 </command_interface>
                 <state_interface name="position"/>
@@ -49,6 +49,6 @@
             <joint name="forearm_hand_2_joint">
                 <command_interface name="position">
-                <param name="min">-${2*pi/3}</param>
-                <param name="max">${2*pi/3}</param>
+                <param name="min">-${2*PI/3}</param>
+                <param name="max">${2*PI/3}</param>
                 </command_interface>
                 <state_interface name="position"/>
@@ -56,6 +56,6 @@
             <joint name="forearm_hand_3_joint">
                 <command_interface name="position">
-                <param name="min">-${2*pi/3}</param>
-                <param name="max">${2*pi/3}</param>
+                <param name="min">-${2*PI/3}</param>
+                <param name="max">${2*PI/3}</param>
                 </command_interface>
                 <state_interface name="position"/>
@@ -63,6 +63,6 @@
              <joint name="forearm_claw_joint">
                 <command_interface name="position">
-                <param name="min">-${2*pi/3}</param>
-                <param name="max">${2*pi/3}</param>
+                <param name="min">-${2*PI/3}</param>
+                <param name="max">${2*PI/3}</param>
                 </command_interface>
                 <state_interface name="position"/>
@@ -70,6 +70,6 @@
             <joint name="joint_4">
                 <command_interface name="position">
-                <param name="min">-${pi / 2}</param>
-                <param name="max">${pi / 2}</param>
+                <param name="min">-${PI / 2}</param>
+                <param name="max">${PI / 2}</param>
                 </command_interface>
                 <state_interface name="position"/>
@@ -80,5 +80,5 @@
                 <command_interface name="position">
                 <param name="min">0.0</param>
-                <param name="max">${pi / 2}</param>
+                <param name="max">${PI / 2}</param>
                 </command_interface>
             </joint> -->
@@ -108,6 +108,6 @@
             <joint name="arm_base_forearm_joint">
                 <command_interface name="position">
-                <param name="min">-${pi / 2}</param>
-                <param name="max">${pi / 2}</param>
+                <param name="min">-${PI / 2}</param>
+                <param name="max">${PI / 2}</param>
                 </command_interface>
                 <state_interface name="position"/>
@@ -117,6 +117,6 @@
             <joint name="forearm_hand_1_joint">
                 <command_interface name="position">
-                <param name="min">-${pi / 2}</param>
-                <param name="max">${pi / 2}</param>
+                <param name="min">-${PI / 2}</param>
+                <param name="max">${PI / 2}</param>
                 </command_interface>
                 <state_interface name="position"/>
@@ -126,6 +126,6 @@
             <joint name="forearm_hand_2_joint">
                 <command_interface name="position">
-                <param name="min">-${pi / 2}</param>
-                <param name="max">${pi / 2}</param>
+                <param name="min">-${PI / 2}</param>
+                <param name="max">${PI / 2}</param>
                 </command_interface>
                 <state_interface name="position"/>
@@ -135,6 +135,6 @@
             <joint name="forearm_hand_3_joint">
                 <command_interface name="position">
-                <param name="min">-${pi / 2}</param>
-                <param name="max">${pi / 2}</param>
+                <param name="min">-${PI / 2}</param>
+                <param name="max">${PI / 2}</param>
                 </command_interface>
                 <state_interface name="position"/>
@@ -144,6 +144,6 @@
              <joint name="forearm_claw_joint">
                 <command_interface name="position">
-                <param name="min">-${pi / 2}</param>
-                <param name="max">${pi / 2}</param>
+                <param name="min">-${PI / 2}</param>
+                <param name="max">${PI / 2}</param>
                 </command_interface>
                 <state_interface name="position"/>
@@ -153,5 +153,5 @@
             <joint name="joint_4">
                 <command_interface name="position">
-                <param name="min">-${pi / 2}</param>
+                <param name="min">-${PI / 2}</param>
                 <param name="max">0.0</param>
                 </command_interface>
@@ -165,5 +165,5 @@
                 <command_interface name="position">
                 <param name="min">0.0</param>
-                <param name="max">${pi / 2}</param>
+                <param name="max">${PI / 2}</param>
                 </command_interface>
                 <state_interface name="position"/>
