Commit message: 31

File: src/articubot_one/description/arm_robot.xacro (robot description, xacro)
@@ -182,5 +182,5 @@
         <child link="hand_2_link" />
         <origin xyz="0 0 ${hand_length}" rpy="0 0 0" />
-        <axis xyz="0 1 0" />
+        <axis xyz="0 -1 0" />
         <limit lower="${-pi/2}" upper="${pi/2}" effort="100" velocity="100" />
         <dynamics friction="0.05" damping="0.1" />
@@ -190,5 +190,5 @@
         <child link="hand_3_link" />
         <origin xyz="0 0 ${hand_length}" rpy="0 0 0" />
-        <axis xyz="0 1 0" />
+        <axis xyz="0 -1 0" />
         <limit lower="${-pi/2}" upper="${pi/2}" effort="100" velocity="100" />
         <dynamics friction="0.05" damping="0.1" />

Commit message: 3132

File: src/articubot_one/description/arm_robot.xacro (robot description, xacro)
@@ -167,5 +167,5 @@
         <origin xyz="0 0 ${arm_base_height}" rpy="0 0 0" />
         <axis xyz="0 0 1" />
-        <limit lower="${-pi/2}" upper="${pi/2}" effort="100" velocity="100" />
+        <limit lower="${-pi}" upper="${pi}" effort="100" velocity="100" />
         <dynamics friction="0.05" damping="0.1" />
     </joint>
@@ -183,5 +183,5 @@
         <origin xyz="0 0 ${hand_length}" rpy="0 0 0" />
         <axis xyz="0 -1 0" />
-        <limit lower="${-pi/2}" upper="${pi/2}" effort="100" velocity="100" />
+        <limit lower="${-pi}" upper="${pi}" effort="100" velocity="100" />
         <dynamics friction="0.05" damping="0.1" />
     </joint>
@@ -191,5 +191,5 @@
         <origin xyz="0 0 ${hand_length}" rpy="0 0 0" />
         <axis xyz="0 -1 0" />
-        <limit lower="${-pi/2}" upper="${pi/2}" effort="100" velocity="100" />
+        <limit lower="${-pi}" upper="${pi}" effort="100" velocity="100" />
         <dynamics friction="0.05" damping="0.1" />
     </joint>

Commit message: 312

File: src/articubot_one/description/arm_robot.xacro (robot description, xacro)
@@ -207,5 +207,5 @@
         <origin xyz="0 0.05 ${hand_length/8}"/>
         <axis xyz="1 0 0"/>
-        <limit lower="-${PI / 2}" upper="0.0"
+        <limit lower="-${PI}" upper="${PI}"
                effort="100" velocity="100"/>
     </joint>
@@ -215,5 +215,5 @@
         <origin xyz="0 -.05 ${hand_length/8}"/>
         <axis xyz="1 0 0"/>
-        <limit lower="0.0" upper="${PI / 2}"
+        <limit lower="-${PI}" upper="${PI}"
                effort="100" velocity="100"/>
         <mimic joint="joint_4" multiplier="-1"/>

Commit message: 312

File: src/articubot_one/description/arm_robot.xacro (robot description, xacro)
@@ -167,5 +167,5 @@
         <origin xyz="0 0 ${arm_base_height}" rpy="0 0 0" />
         <axis xyz="0 0 1" />
-        <limit lower="${-pi}" upper="${pi}" effort="100" velocity="100" />
+        <limit lower="${0.0}" upper="${2*pi}" effort="100" velocity="100" />
         <dynamics friction="0.05" damping="0.1" />
     </joint>
@@ -175,5 +175,5 @@
         <origin xyz="0 0 ${forearm_length}" rpy="0 0 0" />
         <axis xyz="0 1 0" />
-        <limit lower="${-pi}" upper="${pi}" effort="100" velocity="100" />
+        <limit lower="${0.0}" upper="${2*pi}" effort="100" velocity="100" />
         <dynamics friction="0.05" damping="0.1" />
     </joint>
@@ -183,5 +183,5 @@
         <origin xyz="0 0 ${hand_length}" rpy="0 0 0" />
         <axis xyz="0 -1 0" />
-        <limit lower="${-pi}" upper="${pi}" effort="100" velocity="100" />
+        <limit lower="${0.0}" upper="${2*pi}" effort="100" velocity="100" />
         <dynamics friction="0.05" damping="0.1" />
     </joint>
@@ -191,5 +191,5 @@
         <origin xyz="0 0 ${hand_length}" rpy="0 0 0" />
         <axis xyz="0 -1 0" />
-        <limit lower="${-pi}" upper="${pi}" effort="100" velocity="100" />
+        <limit lower="${0.0}" upper="${2*pi}" effort="100" velocity="100" />
         <dynamics friction="0.05" damping="0.1" />
     </joint>
@@ -199,5 +199,5 @@
         <origin xyz="0 0 ${hand_length}" rpy="0 0 0" />
         <axis xyz="0 0 1" />
-        <limit lower="${-pi}" upper="${pi}" effort="100" velocity="100" />
+        <limit lower="${0.0}" upper="${2*pi}" effort="100" velocity="100" />
         <dynamics friction="0.05" damping="0.1" />
     </joint>

Commit message: 312

File: src/articubot_one/description/arm_robot.xacro (robot description, xacro)
@@ -167,5 +167,5 @@
         <origin xyz="0 0 ${arm_base_height}" rpy="0 0 0" />
         <axis xyz="0 0 1" />
-        <limit lower="${0.0}" upper="${2*pi}" effort="100" velocity="100" />
+        <limit lower="${-pi/2}" upper="${pi/2}" effort="100" velocity="100" />
         <dynamics friction="0.05" damping="0.1" />
     </joint>
@@ -175,5 +175,5 @@
         <origin xyz="0 0 ${forearm_length}" rpy="0 0 0" />
         <axis xyz="0 1 0" />
-        <limit lower="${0.0}" upper="${2*pi}" effort="100" velocity="100" />
+        <limit lower="${-pi}" upper="${pi}" effort="100" velocity="100" />
         <dynamics friction="0.05" damping="0.1" />
     </joint>
@@ -183,5 +183,5 @@
         <origin xyz="0 0 ${hand_length}" rpy="0 0 0" />
         <axis xyz="0 -1 0" />
-        <limit lower="${0.0}" upper="${2*pi}" effort="100" velocity="100" />
+        <limit lower="${-pi/2}" upper="${pi/2}" effort="100" velocity="100" />
         <dynamics friction="0.05" damping="0.1" />
     </joint>
@@ -191,5 +191,5 @@
         <origin xyz="0 0 ${hand_length}" rpy="0 0 0" />
         <axis xyz="0 -1 0" />
-        <limit lower="${0.0}" upper="${2*pi}" effort="100" velocity="100" />
+        <limit lower="${-pi/2}" upper="${pi/2}" effort="100" velocity="100" />
         <dynamics friction="0.05" damping="0.1" />
     </joint>
@@ -199,5 +199,5 @@
         <origin xyz="0 0 ${hand_length}" rpy="0 0 0" />
         <axis xyz="0 0 1" />
-        <limit lower="${0.0}" upper="${2*pi}" effort="100" velocity="100" />
+        <limit lower="${-pi}" upper="${pi}" effort="100" velocity="100" />
         <dynamics friction="0.05" damping="0.1" />
     </joint>
@@ -207,5 +207,5 @@
         <origin xyz="0 0.05 ${hand_length/8}"/>
         <axis xyz="1 0 0"/>
-        <limit lower="-${PI}" upper="${PI}"
+        <limit lower="-${PI / 2}" upper="0.0"
                effort="100" velocity="100"/>
     </joint>
@@ -215,5 +215,5 @@
         <origin xyz="0 -.05 ${hand_length/8}"/>
         <axis xyz="1 0 0"/>
-        <limit lower="-${PI}" upper="${PI}"
+        <limit lower="0.0" upper="${PI / 2}"
                effort="100" velocity="100"/>
         <mimic joint="joint_4" multiplier="-1"/>

Commit message: 312

File: src/articubot_one/description/arm_robot.xacro (robot description, xacro)
@@ -175,5 +175,5 @@
         <origin xyz="0 0 ${forearm_length}" rpy="0 0 0" />
         <axis xyz="0 1 0" />
-        <limit lower="${-pi}" upper="${pi}" effort="100" velocity="100" />
+        <limit lower="${-pi/2}" upper="${pi/2}" effort="100" velocity="100" />
         <dynamics friction="0.05" damping="0.1" />
     </joint>
@@ -199,5 +199,5 @@
         <origin xyz="0 0 ${hand_length}" rpy="0 0 0" />
         <axis xyz="0 0 1" />
-        <limit lower="${-pi}" upper="${pi}" effort="100" velocity="100" />
+        <limit lower="${-pi/2}" upper="${pi/2}" effort="100" velocity="100" />
         <dynamics friction="0.05" damping="0.1" />
     </joint>

Commit message: 31

File: src/articubot_one/description/arm_robot.xacro (robot description, xacro)
@@ -182,5 +182,5 @@
         <child link="hand_2_link" />
         <origin xyz="0 0 ${hand_length}" rpy="0 0 0" />
-        <axis xyz="0 -1 0" />
+        <axis xyz="0 1 0" />
         <limit lower="${-pi/2}" upper="${pi/2}" effort="100" velocity="100" />
         <dynamics friction="0.05" damping="0.1" />

Commit message: 312

File: src/articubot_one/description/arm_robot.xacro (robot description, xacro)
@@ -174,5 +174,5 @@
         <child link="hand_1_link" />
         <origin xyz="0 0 ${forearm_length}" rpy="0 0 0" />
-        <axis xyz="0 1 0" />
+        <axis xyz="0 -1 0" />
         <limit lower="${-pi/2}" upper="${pi/2}" effort="100" velocity="100" />
         <dynamics friction="0.05" damping="0.1" />
@@ -182,5 +182,5 @@
         <child link="hand_2_link" />
         <origin xyz="0 0 ${hand_length}" rpy="0 0 0" />
-        <axis xyz="0 1 0" />
+        <axis xyz="0 -1 0" />
         <limit lower="${-pi/2}" upper="${pi/2}" effort="100" velocity="100" />
         <dynamics friction="0.05" damping="0.1" />

Commit message: 312

File: src/articubot_one/description/arm_robot.xacro (robot description, xacro)
@@ -175,5 +175,5 @@
         <origin xyz="0 0 ${forearm_length}" rpy="0 0 0" />
         <axis xyz="0 -1 0" />
-        <limit lower="${-pi/2}" upper="${pi/2}" effort="100" velocity="100" />
+        <limit lower="${0.0}" upper="${pi}" effort="100" velocity="100" />
         <dynamics friction="0.05" damping="0.1" />
     </joint>

Commit message: 312

File: src/articubot_one/description/arm_robot.xacro (robot description, xacro)
@@ -175,5 +175,5 @@
         <origin xyz="0 0 ${forearm_length}" rpy="0 0 0" />
         <axis xyz="0 -1 0" />
-        <limit lower="${0.0}" upper="${pi}" effort="100" velocity="100" />
+        <limit lower="${-pi}" upper="${0.0}" effort="100" velocity="100" />
         <dynamics friction="0.05" damping="0.1" />
     </joint>

Commit message: 31

File: src/articubot_one/description/arm_robot.xacro (robot description, xacro)
@@ -175,5 +175,5 @@
         <origin xyz="0 0 ${forearm_length}" rpy="0 0 0" />
         <axis xyz="0 -1 0" />
-        <limit lower="${-pi}" upper="${0.0}" effort="100" velocity="100" />
+        <limit lower="${-pi/2}" upper="${pi/2}" effort="100" velocity="100" />
         <dynamics friction="0.05" damping="0.1" />
     </joint>

Commit message: 312

File: src/articubot_one/description/arm_robot.xacro (robot description, xacro)
@@ -174,6 +174,6 @@
         <child link="hand_1_link" />
         <origin xyz="0 0 ${forearm_length}" rpy="0 0 0" />
-        <axis xyz="0 -1 0" />
-        <limit lower="${-pi/2}" upper="${pi/2}" effort="100" velocity="100" />
+        <axis xyz="0 1 0" />
+        <limit lower="${pi/2}" upper="${-pi/2}" effort="100" velocity="100" />
         <dynamics friction="0.05" damping="0.1" />
     </joint>

File: src/articubot_one/description/ros2_control.xacro (robot description, xacro)
@@ -39,6 +39,6 @@
             <joint name="forearm_hand_1_joint">
                 <command_interface name="position">
-                <param name="min">-${PI / 2}</param>
-                <param name="max">${PI / 2}</param>
+                <param name="min">${PI / 2}</param>
+                <param name="max">-${PI / 2}</param>
                 </command_interface>
                 <state_interface name="position"/>

Commit message: 31

File: src/articubot_one/description/arm_robot.xacro (robot description, xacro)
@@ -174,5 +174,5 @@
         <child link="hand_1_link" />
         <origin xyz="0 0 ${forearm_length}" rpy="0 0 0" />
-        <axis xyz="0 1 0" />
+        <axis xyz="0 -1 0" />
         <limit lower="${pi/2}" upper="${-pi/2}" effort="100" velocity="100" />
         <dynamics friction="0.05" damping="0.1" />

Commit message: 312

File: src/articubot_one/description/arm_robot.xacro (robot description, xacro)
@@ -174,6 +174,6 @@
         <child link="hand_1_link" />
         <origin xyz="0 0 ${forearm_length}" rpy="0 0 0" />
-        <axis xyz="0 -1 0" />
-        <limit lower="${pi/2}" upper="${-pi/2}" effort="100" velocity="100" />
+        <axis xyz="0 1 0" />
+        <limit lower="${-pi/2}" upper="${pi/2}" effort="100" velocity="100" />
         <dynamics friction="0.05" damping="0.1" />
     </joint>

File: src/articubot_one/description/ros2_control.xacro (robot description, xacro)
@@ -39,6 +39,6 @@
             <joint name="forearm_hand_1_joint">
                 <command_interface name="position">
-                <param name="min">${PI / 2}</param>
-                <param name="max">-${PI / 2}</param>
+                <param name="min">-${PI / 2}</param>
+                <param name="max">${PI / 2}</param>
                 </command_interface>
                 <state_interface name="position"/>

Commit message: 31

File: src/articubot_one/description/arm_robot.xacro (robot description, xacro)
@@ -174,5 +174,5 @@
         <child link="hand_1_link" />
         <origin xyz="0 0 ${forearm_length}" rpy="0 0 0" />
-        <axis xyz="0 1 0" />
+        <axis xyz="0 -1 0" />
         <limit lower="${-pi/2}" upper="${pi/2}" effort="100" velocity="100" />
         <dynamics friction="0.05" damping="0.1" />

Commit message: 312

File: src/articubot_one/description/arm_robot.xacro (robot description, xacro)
@@ -175,5 +175,5 @@
         <origin xyz="0 0 ${forearm_length}" rpy="0 0 0" />
         <axis xyz="0 -1 0" />
-        <limit lower="${-pi/2}" upper="${pi/2}" effort="100" velocity="100" />
+        <limit lower="${pi/2}" upper="${-pi/2}" effort="100" velocity="100" />
         <dynamics friction="0.05" damping="0.1" />
     </joint>

Commit message: 312

File: src/articubot_one/description/arm_robot.xacro (robot description, xacro)
@@ -175,5 +175,5 @@
         <origin xyz="0 0 ${forearm_length}" rpy="0 0 0" />
         <axis xyz="0 -1 0" />
-        <limit lower="${pi/2}" upper="${-pi/2}" effort="100" velocity="100" />
+        <limit lower="${-pi/2}" upper="${pi/2}" effort="100" velocity="100" />
         <dynamics friction="0.05" damping="0.1" />
     </joint>

Commit message: 312

File: src/articubot_one/description/arm_robot.xacro (robot description, xacro)
@@ -174,5 +174,5 @@
         <child link="hand_1_link" />
         <origin xyz="0 0 ${forearm_length}" rpy="0 0 0" />
-        <axis xyz="0 -1 0" />
+        <axis xyz="0 1 0" />
         <limit lower="${-pi/2}" upper="${pi/2}" effort="100" velocity="100" />
         <dynamics friction="0.05" damping="0.1" />

Commit message: 323

File: src/articubot_one/description/arm_robot.xacro (robot description, xacro)
@@ -182,5 +182,5 @@
         <child link="hand_2_link" />
         <origin xyz="0 0 ${hand_length}" rpy="0 0 0" />
-        <axis xyz="0 1 0" />
+        <axis xyz="0 -1 0" />
         <limit lower="${-pi/2}" upper="${pi/2}" effort="100" velocity="100" />
         <dynamics friction="0.05" damping="0.1" />

Commit message: 232

File: src/articubot_one/description/arm_robot.xacro (robot description, xacro)
@@ -207,5 +207,5 @@
         <origin xyz="0 0.05 ${hand_length/8}"/>
         <axis xyz="1 0 0"/>
-        <limit lower="-${PI / 2}" upper="0.0"
+        <limit lower="-${PI / 2}" upper="${PI / 2}"
                effort="100" velocity="100"/>
     </joint>

File: src/articubot_one/description/ros2_control.xacro (robot description, xacro)
@@ -68,5 +68,5 @@
                 <command_interface name="position">
                 <param name="min">-${PI / 2}</param>
-                <param name="max">0.0</param>
+                <param name="max">${PI / 2}</param>
                 </command_interface>
                 <state_interface name="position"/>

Commit message: 13

File: src/articubot_one/description/arm_robot.xacro (robot description, xacro)
@@ -215,5 +215,5 @@
         <origin xyz="0 -.05 ${hand_length/8}"/>
         <axis xyz="1 0 0"/>
-        <limit lower="0.0" upper="${PI / 2}"
+        <limit lower="-${PI / 2}" upper="${PI / 2}"
                effort="100" velocity="100"/>
         <mimic joint="joint_4" multiplier="-1"/>

Commit message: asd

File: src/articubot_one/description/arm_robot.xacro (robot description, xacro)
@@ -167,5 +167,5 @@
         <origin xyz="0 0 ${arm_base_height}" rpy="0 0 0" />
         <axis xyz="0 0 1" />
-        <limit lower="${-pi/2}" upper="${pi/2}" effort="100" velocity="100" />
+        <limit lower="${-pi/2}" upper="${pi/2}" effort="100" velocity="1.0" />
         <dynamics friction="0.05" damping="0.1" />
     </joint>
@@ -175,5 +175,5 @@
         <origin xyz="0 0 ${forearm_length}" rpy="0 0 0" />
         <axis xyz="0 1 0" />
-        <limit lower="${-pi/2}" upper="${pi/2}" effort="100" velocity="100" />
+        <limit lower="${-pi/2}" upper="${pi/2}" effort="100" velocity="1.0" />
         <dynamics friction="0.05" damping="0.1" />
     </joint>
@@ -183,5 +183,5 @@
         <origin xyz="0 0 ${hand_length}" rpy="0 0 0" />
         <axis xyz="0 -1 0" />
-        <limit lower="${-pi/2}" upper="${pi/2}" effort="100" velocity="100" />
+        <limit lower="${-pi/2}" upper="${pi/2}" effort="100" velocity="1.0" />
         <dynamics friction="0.05" damping="0.1" />
     </joint>
@@ -191,5 +191,5 @@
         <origin xyz="0 0 ${hand_length}" rpy="0 0 0" />
         <axis xyz="0 -1 0" />
-        <limit lower="${-pi/2}" upper="${pi/2}" effort="100" velocity="100" />
+        <limit lower="${-pi/2}" upper="${pi/2}" effort="100" velocity="1.0" />
         <dynamics friction="0.05" damping="0.1" />
     </joint>
@@ -199,5 +199,5 @@
         <origin xyz="0 0 ${hand_length}" rpy="0 0 0" />
         <axis xyz="0 0 1" />
-        <limit lower="${-pi/2}" upper="${pi/2}" effort="100" velocity="100" />
+        <limit lower="${-pi/2}" upper="${pi/2}" effort="100" velocity="1.0" />
         <dynamics friction="0.05" damping="0.1" />
     </joint>

Commit message: 31

File: src/articubot_one/description/arm_robot.xacro (robot description, xacro)
@@ -167,5 +167,5 @@
         <origin xyz="0 0 ${arm_base_height}" rpy="0 0 0" />
         <axis xyz="0 0 1" />
-        <limit lower="${-pi/2}" upper="${pi/2}" effort="100" velocity="1.0" />
+        <limit lower="${-pi/2}" upper="${pi/2}" effort="100" velocity="10.0" />
         <dynamics friction="0.05" damping="0.1" />
     </joint>
@@ -175,5 +175,5 @@
         <origin xyz="0 0 ${forearm_length}" rpy="0 0 0" />
         <axis xyz="0 1 0" />
-        <limit lower="${-pi/2}" upper="${pi/2}" effort="100" velocity="1.0" />
+        <limit lower="${-pi/2}" upper="${pi/2}" effort="100" velocity="10.0" />
         <dynamics friction="0.05" damping="0.1" />
     </joint>
@@ -183,5 +183,5 @@
         <origin xyz="0 0 ${hand_length}" rpy="0 0 0" />
         <axis xyz="0 -1 0" />
-        <limit lower="${-pi/2}" upper="${pi/2}" effort="100" velocity="1.0" />
+        <limit lower="${-pi/2}" upper="${pi/2}" effort="100" velocity="10.0" />
         <dynamics friction="0.05" damping="0.1" />
     </joint>
@@ -191,5 +191,5 @@
         <origin xyz="0 0 ${hand_length}" rpy="0 0 0" />
         <axis xyz="0 -1 0" />
-        <limit lower="${-pi/2}" upper="${pi/2}" effort="100" velocity="1.0" />
+        <limit lower="${-pi/2}" upper="${pi/2}" effort="100" velocity="10.0" />
         <dynamics friction="0.05" damping="0.1" />
     </joint>
@@ -199,5 +199,5 @@
         <origin xyz="0 0 ${hand_length}" rpy="0 0 0" />
         <axis xyz="0 0 1" />
-        <limit lower="${-pi/2}" upper="${pi/2}" effort="100" velocity="1.0" />
+        <limit lower="${-pi/2}" upper="${pi/2}" effort="100" velocity="10.0" />
         <dynamics friction="0.05" damping="0.1" />
     </joint>

Commit message: 312

File: src/articubot_one/description/arm_robot.xacro (robot description, xacro)
@@ -167,5 +167,5 @@
         <origin xyz="0 0 ${arm_base_height}" rpy="0 0 0" />
         <axis xyz="0 0 1" />
-        <limit lower="${-pi/2}" upper="${pi/2}" effort="100" velocity="10.0" />
+        <limit lower="${-pi/2}" upper="${pi/2}" effort="100" velocity="5.0" />
         <dynamics friction="0.05" damping="0.1" />
     </joint>
@@ -175,5 +175,5 @@
         <origin xyz="0 0 ${forearm_length}" rpy="0 0 0" />
         <axis xyz="0 1 0" />
-        <limit lower="${-pi/2}" upper="${pi/2}" effort="100" velocity="10.0" />
+        <limit lower="${-pi/2}" upper="${pi/2}" effort="100" velocity="5.0" />
         <dynamics friction="0.05" damping="0.1" />
     </joint>
@@ -183,5 +183,5 @@
         <origin xyz="0 0 ${hand_length}" rpy="0 0 0" />
         <axis xyz="0 -1 0" />
-        <limit lower="${-pi/2}" upper="${pi/2}" effort="100" velocity="10.0" />
+        <limit lower="${-pi/2}" upper="${pi/2}" effort="100" velocity="5.0" />
         <dynamics friction="0.05" damping="0.1" />
     </joint>
@@ -191,5 +191,5 @@
         <origin xyz="0 0 ${hand_length}" rpy="0 0 0" />
         <axis xyz="0 -1 0" />
-        <limit lower="${-pi/2}" upper="${pi/2}" effort="100" velocity="10.0" />
+        <limit lower="${-pi/2}" upper="${pi/2}" effort="100" velocity="5.0" />
         <dynamics friction="0.05" damping="0.1" />
     </joint>
@@ -199,5 +199,5 @@
         <origin xyz="0 0 ${hand_length}" rpy="0 0 0" />
         <axis xyz="0 0 1" />
-        <limit lower="${-pi/2}" upper="${pi/2}" effort="100" velocity="10.0" />
+        <limit lower="${-pi/2}" upper="${pi/2}" effort="100" velocity="5.0" />
         <dynamics friction="0.05" damping="0.1" />
     </joint>
@@ -208,5 +208,5 @@
         <axis xyz="1 0 0"/>
         <limit lower="-${PI / 2}" upper="${PI / 2}"
-               effort="100" velocity="10.0"/>
+               effort="100" velocity="5.0"/>
     </joint>
     <joint name ="joint_5" type="revolute">
@@ -216,5 +216,5 @@
         <axis xyz="1 0 0"/>
         <limit lower="-${PI / 2}" upper="${PI / 2}"
-               effort="100" velocity="10.0"/>
+               effort="100" velocity="5.0"/>
         <mimic joint="joint_4" multiplier="-1"/>
     </joint>
