Commit message: 31

File: src/articubot_one/description/arm_robot.xacro (robot description, xacro)
@@ -167,5 +167,5 @@
         <origin xyz="0 0 ${arm_base_height}" rpy="0 0 0" />
         <axis xyz="0 0 1" />
-        <limit lower="${-pi/2}" upper="${pi/2}" effort="100" velocity="5.0" />
+        <limit lower="${-pi/2}" upper="${pi/2}" effort="50" velocity="5.0" />
         <dynamics friction="0.05" damping="0.1" />
     </joint>
@@ -175,5 +175,5 @@
         <origin xyz="0 0 ${forearm_length}" rpy="0 0 0" />
         <axis xyz="0 1 0" />
-        <limit lower="${-pi/2}" upper="${pi/2}" effort="100" velocity="5.0" />
+        <limit lower="${-pi/2}" upper="${pi/2}" effort="50" velocity="5.0" />
         <dynamics friction="0.05" damping="0.1" />
     </joint>
@@ -183,5 +183,5 @@
         <origin xyz="0 0 ${hand_length}" rpy="0 0 0" />
         <axis xyz="0 -1 0" />
-        <limit lower="${-pi/2}" upper="${pi/2}" effort="100" velocity="5.0" />
+        <limit lower="${-pi/2}" upper="${pi/2}" effort="50" velocity="5.0" />
         <dynamics friction="0.05" damping="0.1" />
     </joint>
@@ -191,5 +191,5 @@
         <origin xyz="0 0 ${hand_length}" rpy="0 0 0" />
         <axis xyz="0 -1 0" />
-        <limit lower="${-pi/2}" upper="${pi/2}" effort="100" velocity="5.0" />
+        <limit lower="${-pi/2}" upper="${pi/2}" effort="50" velocity="5.0" />
         <dynamics friction="0.05" damping="0.1" />
     </joint>
@@ -199,5 +199,5 @@
         <origin xyz="0 0 ${hand_length}" rpy="0 0 0" />
         <axis xyz="0 0 1" />
-        <limit lower="${-pi/2}" upper="${pi/2}" effort="100" velocity="5.0" />
+        <limit lower="${-pi/2}" upper="${pi/2}" effort="50" velocity="5.0" />
         <dynamics friction="0.05" damping="0.1" />
     </joint>
@@ -208,5 +208,5 @@
         <axis xyz="1 0 0"/>
         <limit lower="-${PI / 2}" upper="${PI / 2}"
-               effort="100" velocity="5.0"/>
+               effort="50" velocity="5.0"/>
     </joint>
     <joint name ="joint_5" type="revolute">
@@ -216,5 +216,5 @@
         <axis xyz="1 0 0"/>
         <limit lower="-${PI / 2}" upper="${PI / 2}"
-               effort="100" velocity="5.0"/>
+               effort="50" velocity="5.0"/>
         <mimic joint="joint_4" multiplier="-1"/>
     </joint>

Commit message: 32

File: src/articubot_one/description/arm_robot.xacro (robot description, xacro)
@@ -167,5 +167,5 @@
         <origin xyz="0 0 ${arm_base_height}" rpy="0 0 0" />
         <axis xyz="0 0 1" />
-        <limit lower="${-pi/2}" upper="${pi/2}" effort="50" velocity="5.0" />
+        <limit lower="${-pi/2}" upper="${pi/2}" effort="10" velocity="5.0" />
         <dynamics friction="0.05" damping="0.1" />
     </joint>
@@ -175,5 +175,5 @@
         <origin xyz="0 0 ${forearm_length}" rpy="0 0 0" />
         <axis xyz="0 1 0" />
-        <limit lower="${-pi/2}" upper="${pi/2}" effort="50" velocity="5.0" />
+        <limit lower="${-pi/2}" upper="${pi/2}" effort="10" velocity="5.0" />
         <dynamics friction="0.05" damping="0.1" />
     </joint>
@@ -183,5 +183,5 @@
         <origin xyz="0 0 ${hand_length}" rpy="0 0 0" />
         <axis xyz="0 -1 0" />
-        <limit lower="${-pi/2}" upper="${pi/2}" effort="50" velocity="5.0" />
+        <limit lower="${-pi/2}" upper="${pi/2}" effort="10" velocity="5.0" />
         <dynamics friction="0.05" damping="0.1" />
     </joint>
@@ -191,5 +191,5 @@
         <origin xyz="0 0 ${hand_length}" rpy="0 0 0" />
         <axis xyz="0 -1 0" />
-        <limit lower="${-pi/2}" upper="${pi/2}" effort="50" velocity="5.0" />
+        <limit lower="${-pi/2}" upper="${pi/2}" effort="10" velocity="5.0" />
         <dynamics friction="0.05" damping="0.1" />
     </joint>
@@ -199,5 +199,5 @@
         <origin xyz="0 0 ${hand_length}" rpy="0 0 0" />
         <axis xyz="0 0 1" />
-        <limit lower="${-pi/2}" upper="${pi/2}" effort="50" velocity="5.0" />
+        <limit lower="${-pi/2}" upper="${pi/2}" effort="10" velocity="5.0" />
         <dynamics friction="0.05" damping="0.1" />
     </joint>

Commit message: 34

File: src/articubot_one/description/arm_robot.xacro (robot description, xacro)
@@ -168,5 +168,5 @@
         <axis xyz="0 0 1" />
         <limit lower="${-pi/2}" upper="${pi/2}" effort="10" velocity="5.0" />
-        <dynamics friction="0.05" damping="0.1" />
+        <dynamics friction="0.01" damping="0.01" />
     </joint>
     <joint name="forearm_hand_1_joint" type="revolute">
@@ -176,5 +176,5 @@
         <axis xyz="0 1 0" />
         <limit lower="${-pi/2}" upper="${pi/2}" effort="10" velocity="5.0" />
-        <dynamics friction="0.05" damping="0.1" />
+        <dynamics friction="0.01" damping="0.01" />
     </joint>
     <joint name="forearm_hand_2_joint" type="revolute">
@@ -184,5 +184,5 @@
         <axis xyz="0 -1 0" />
         <limit lower="${-pi/2}" upper="${pi/2}" effort="10" velocity="5.0" />
-        <dynamics friction="0.05" damping="0.1" />
+        <dynamics friction="0.01" damping="0.01" />
     </joint>
     <joint name="forearm_hand_3_joint" type="revolute">
@@ -192,5 +192,5 @@
         <axis xyz="0 -1 0" />
         <limit lower="${-pi/2}" upper="${pi/2}" effort="10" velocity="5.0" />
-        <dynamics friction="0.05" damping="0.1" />
+        <dynamics friction="0.01" damping="0.01" />
     </joint>
     <joint name="forearm_claw_joint" type="revolute">
@@ -200,5 +200,5 @@
         <axis xyz="0 0 1" />
         <limit lower="${-pi/2}" upper="${pi/2}" effort="10" velocity="5.0" />
-        <dynamics friction="0.05" damping="0.1" />
+        <dynamics friction="0.01" damping="0.01" />
     </joint>
     <joint name ="joint_4" type="revolute">

Commit message: 32

File: src/articubot_one/description/arm_robot.xacro (robot description, xacro)
@@ -167,5 +167,5 @@
         <origin xyz="0 0 ${arm_base_height}" rpy="0 0 0" />
         <axis xyz="0 0 1" />
-        <limit lower="${-pi/2}" upper="${pi/2}" effort="10" velocity="5.0" />
+        <limit lower="${-pi}" upper="${pi}" effort="10" velocity="5.0" />
         <dynamics friction="0.01" damping="0.01" />
     </joint>
@@ -175,5 +175,5 @@
         <origin xyz="0 0 ${forearm_length}" rpy="0 0 0" />
         <axis xyz="0 1 0" />
-        <limit lower="${-pi/2}" upper="${pi/2}" effort="10" velocity="5.0" />
+        <limit lower="${-pi}" upper="${pi}" effort="10" velocity="5.0" />
         <dynamics friction="0.01" damping="0.01" />
     </joint>
@@ -183,5 +183,5 @@
         <origin xyz="0 0 ${hand_length}" rpy="0 0 0" />
         <axis xyz="0 -1 0" />
-        <limit lower="${-pi/2}" upper="${pi/2}" effort="10" velocity="5.0" />
+        <limit lower="${-pi}" upper="${pi}" effort="10" velocity="5.0" />
         <dynamics friction="0.01" damping="0.01" />
     </joint>
@@ -191,5 +191,5 @@
         <origin xyz="0 0 ${hand_length}" rpy="0 0 0" />
         <axis xyz="0 -1 0" />
-        <limit lower="${-pi/2}" upper="${pi/2}" effort="10" velocity="5.0" />
+        <limit lower="${-pi}" upper="${pi}" effort="10" velocity="5.0" />
         <dynamics friction="0.01" damping="0.01" />
     </joint>
@@ -199,5 +199,5 @@
         <origin xyz="0 0 ${hand_length}" rpy="0 0 0" />
         <axis xyz="0 0 1" />
-        <limit lower="${-pi/2}" upper="${pi/2}" effort="10" velocity="5.0" />
+        <limit lower="${-pi}" upper="${pi}" effort="10" velocity="5.0" />
         <dynamics friction="0.01" damping="0.01" />
     </joint>

Commit message: 32

File: src/articubot_one/description/arm_robot.xacro (robot description, xacro)
@@ -167,5 +167,5 @@
         <origin xyz="0 0 ${arm_base_height}" rpy="0 0 0" />
         <axis xyz="0 0 1" />
-        <limit lower="${-pi}" upper="${pi}" effort="10" velocity="5.0" />
+        <limit lower="${-pi/2}" upper="${pi/2}" effort="10" velocity="5.0" />
         <dynamics friction="0.01" damping="0.01" />
     </joint>
@@ -175,5 +175,5 @@
         <origin xyz="0 0 ${forearm_length}" rpy="0 0 0" />
         <axis xyz="0 1 0" />
-        <limit lower="${-pi}" upper="${pi}" effort="10" velocity="5.0" />
+        <limit lower="${-pi/2}" upper="${pi/2}" effort="10" velocity="5.0" />
         <dynamics friction="0.01" damping="0.01" />
     </joint>
@@ -183,5 +183,5 @@
         <origin xyz="0 0 ${hand_length}" rpy="0 0 0" />
         <axis xyz="0 -1 0" />
-        <limit lower="${-pi}" upper="${pi}" effort="10" velocity="5.0" />
+        <limit lower="${-pi/2}" upper="${pi/2}" effort="10" velocity="5.0" />
         <dynamics friction="0.01" damping="0.01" />
     </joint>
@@ -191,5 +191,5 @@
         <origin xyz="0 0 ${hand_length}" rpy="0 0 0" />
         <axis xyz="0 -1 0" />
-        <limit lower="${-pi}" upper="${pi}" effort="10" velocity="5.0" />
+        <limit lower="${-pi/2}" upper="${pi/2}" effort="10" velocity="5.0" />
         <dynamics friction="0.01" damping="0.01" />
     </joint>
@@ -199,5 +199,5 @@
         <origin xyz="0 0 ${hand_length}" rpy="0 0 0" />
         <axis xyz="0 0 1" />
-        <limit lower="${-pi}" upper="${pi}" effort="10" velocity="5.0" />
+        <limit lower="${-pi/2}" upper="${pi/2}" effort="10" velocity="5.0" />
         <dynamics friction="0.01" damping="0.01" />
     </joint>

File: src/articubot_one/description/ros2_control.xacro (robot description, xacro)
@@ -35,6 +35,6 @@
             <joint name="arm_base_forearm_joint">
                 <command_interface name="position">
-                <param name="min">-${PI}</param>
-                <param name="max">${PI}</param>
+                <param name="min">-${PI/2}</param>
+                <param name="max">${PI/2}</param>
                 </command_interface>
                 <state_interface name="position"/>
@@ -42,6 +42,6 @@
             <joint name="forearm_hand_1_joint">
                 <command_interface name="position">
-                <param name="min">-${PI}</param>
-                <param name="max">${PI}</param>
+                <param name="min">-${PI/2}</param>
+                <param name="max">${PI/2}</param>
                 </command_interface>
                 <state_interface name="position"/>
@@ -49,6 +49,6 @@
             <joint name="forearm_hand_2_joint">
                 <command_interface name="position">
-                <param name="min">-${PI}</param>
-                <param name="max">${PI}</param>
+                <param name="min">-${PI/2}</param>
+                <param name="max">${PI/2}</param>
                 </command_interface>
                 <state_interface name="position"/>
@@ -56,6 +56,6 @@
             <joint name="forearm_hand_3_joint">
                 <command_interface name="position">
-                <param name="min">-${PI}</param>
-                <param name="max">${PI}</param>
+                <param name="min">-${PI/2}</param>
+                <param name="max">${PI/2}</param>
                 </command_interface>
                 <state_interface name="position"/>
@@ -63,6 +63,6 @@
              <joint name="forearm_claw_joint">
                 <command_interface name="position">
-                <param name="min">-${PI}</param>
-                <param name="max">${PI}</param>
+                <param name="min">-${PI/2}</param>
+                <param name="max">${PI/2}</param>
                 </command_interface>
                 <state_interface name="position"/>

Commit message: 3232

File: src/articubot_one/description/arm_robot.xacro (robot description, xacro)
@@ -167,5 +167,5 @@
         <origin xyz="0 0 ${arm_base_height}" rpy="0 0 0" />
         <axis xyz="0 0 1" />
-        <limit lower="${-pi/2}" upper="${pi/2}" effort="10" velocity="5.0" />
+        <limit lower="${-2*PI/3}" upper="${2*PI/3}" effort="10" velocity="5.0" />
         <dynamics friction="0.01" damping="0.01" />
     </joint>
@@ -175,5 +175,5 @@
         <origin xyz="0 0 ${forearm_length}" rpy="0 0 0" />
         <axis xyz="0 1 0" />
-        <limit lower="${-pi/2}" upper="${pi/2}" effort="10" velocity="5.0" />
+        <limit lower="${-2*PI/3}" upper="${2*PI/3}" effort="10" velocity="5.0" />
         <dynamics friction="0.01" damping="0.01" />
     </joint>
@@ -183,5 +183,5 @@
         <origin xyz="0 0 ${hand_length}" rpy="0 0 0" />
         <axis xyz="0 -1 0" />
-        <limit lower="${-pi/2}" upper="${pi/2}" effort="10" velocity="5.0" />
+        <limit lower="${-2*PI/3}" upper="${2*PI/3}" effort="10" velocity="5.0" />
         <dynamics friction="0.01" damping="0.01" />
     </joint>
@@ -191,5 +191,5 @@
         <origin xyz="0 0 ${hand_length}" rpy="0 0 0" />
         <axis xyz="0 -1 0" />
-        <limit lower="${-pi/2}" upper="${pi/2}" effort="10" velocity="5.0" />
+        <limit lower="${-2*PI/3}" upper="${2*PI/3}" effort="10" velocity="5.0" />
         <dynamics friction="0.01" damping="0.01" />
     </joint>
@@ -199,5 +199,5 @@
         <origin xyz="0 0 ${hand_length}" rpy="0 0 0" />
         <axis xyz="0 0 1" />
-        <limit lower="${-pi/2}" upper="${pi/2}" effort="10" velocity="5.0" />
+        <limit lower="${-2*PI/3}" upper="${2*PI/3}" effort="10" velocity="5.0" />
         <dynamics friction="0.01" damping="0.01" />
     </joint>

File: src/articubot_one/description/camera.xacro (robot description, xacro)
@@ -24,5 +24,5 @@
         <parent link="camera_link"/>
         <child link="camera_link_optical"/>
-        <origin xyz="0 0 0" rpy="${-pi/2} 0 ${-pi/2}"/>
+        <origin xyz="0 0 0" rpy="${-PI/2} 0 ${-PI/2}"/>
     </joint>
     <link name="camera_link_optical"></link>

File: src/articubot_one/description/depth_camera.xacro (robot description, xacro)
@@ -23,5 +23,5 @@
         <parent link="camera_link"/>
         <child link="camera_link_optical"/>
-        <origin xyz="0 0 0" rpy="${-pi/2} 0 ${-pi/2}"/>
+        <origin xyz="0 0 0" rpy="${-PI/2} 0 ${-PI/2}"/>
     </joint>
     <link name="camera_link_optical"></link>

File: src/articubot_one/description/face.xacro (robot description, xacro)
@@ -8,5 +8,5 @@
     <link name="face_link">
         <visual>
-            <origin xyz="0 0.05 0.01" rpy="0 ${pi/2} 0"/>
+            <origin xyz="0 0.05 0.01" rpy="0 ${PI/2} 0"/>
             <geometry>
                 <cylinder radius="0.01" length="0.002"/>
@@ -15,5 +15,5 @@
         </visual>
         <visual>
-            <origin xyz="0 -0.05 0.01" rpy="0 ${pi/2} 0"/>
+            <origin xyz="0 -0.05 0.01" rpy="0 ${PI/2} 0"/>
             <geometry>
                 <cylinder radius="0.01" length="0.002"/>

File: src/articubot_one/description/robot_core.xacro (robot description, xacro)
@@ -73,5 +73,5 @@
         <parent link="base_link"/>
         <child link="left_wheel"/>
-        <origin xyz="0 ${wheel_offset_y} 0" rpy="-${pi/2} 0 0" />
+        <origin xyz="0 ${wheel_offset_y} 0" rpy="-${PI/2} 0 0" />
         <axis xyz="0 0 1"/>
     </joint>
@@ -99,5 +99,5 @@
         <parent link="base_link"/>
         <child link="right_wheel"/>
-        <origin xyz="0 ${-wheel_offset_y} 0" rpy="${pi/2} 0 0" />
+        <origin xyz="0 ${-wheel_offset_y} 0" rpy="${PI/2} 0 0" />
         <axis xyz="0 0 -1"/>
     </joint>

File: src/articubot_one/description/ros2_control.xacro (robot description, xacro)
@@ -35,6 +35,6 @@
             <joint name="arm_base_forearm_joint">
                 <command_interface name="position">
-                <param name="min">-${PI/2}</param>
-                <param name="max">${PI/2}</param>
+                <param name="min">-${2*PI/3}</param>
+                <param name="max">${2*PI/3}</param>
                 </command_interface>
                 <state_interface name="position"/>
@@ -42,6 +42,6 @@
             <joint name="forearm_hand_1_joint">
                 <command_interface name="position">
-                <param name="min">-${PI/2}</param>
-                <param name="max">${PI/2}</param>
+                <param name="min">-${2*PI/3}</param>
+                <param name="max">${2*PI/3}</param>
                 </command_interface>
                 <state_interface name="position"/>
@@ -49,6 +49,6 @@
             <joint name="forearm_hand_2_joint">
                 <command_interface name="position">
-                <param name="min">-${PI/2}</param>
-                <param name="max">${PI/2}</param>
+                <param name="min">-${2*PI/3}</param>
+                <param name="max">${2*PI/3}</param>
                 </command_interface>
                 <state_interface name="position"/>
@@ -56,6 +56,6 @@
             <joint name="forearm_hand_3_joint">
                 <command_interface name="position">
-                <param name="min">-${PI/2}</param>
-                <param name="max">${PI/2}</param>
+                <param name="min">-${2*PI/3}</param>
+                <param name="max">${2*PI/3}</param>
                 </command_interface>
                 <state_interface name="position"/>
@@ -63,6 +63,6 @@
              <joint name="forearm_claw_joint">
                 <command_interface name="position">
-                <param name="min">-${PI/2}</param>
-                <param name="max">${PI/2}</param>
+                <param name="min">-${2*PI/3}</param>
+                <param name="max">${2*PI/3}</param>
                 </command_interface>
                 <state_interface name="position"/>
