Commit message: 32

File: src/articubot_one/description/arm_robot.xacro (robot description, xacro)
@@ -18,5 +18,5 @@
         </inertial>
     </xacro:macro>
-    <xacro:property name="PI" value="3.14159265359" />
+    <xacro:property name="pi" value="3.14159265359" />
     <xacro:property name="effort" value="30.0" />
     <xacro:property name="velocity" value="10.0" />
@@ -167,5 +167,5 @@
         <origin xyz="0 0 ${arm_base_height}" rpy="0 0 0" />
         <axis xyz="0 0 1" />
-        <limit lower="${-2*PI/3}" upper="${2*PI/3}" effort="10" velocity="5.0" />
+        <limit lower="${-2*pi/3}" upper="${2*pi/3}" effort="10" velocity="5.0" />
         <dynamics friction="0.01" damping="0.01" />
     </joint>
@@ -175,5 +175,5 @@
         <origin xyz="0 0 ${forearm_length}" rpy="0 0 0" />
         <axis xyz="0 1 0" />
-        <limit lower="${-2*PI/3}" upper="${2*PI/3}" effort="10" velocity="5.0" />
+        <limit lower="${-2*pi/3}" upper="${2*pi/3}" effort="10" velocity="5.0" />
         <dynamics friction="0.01" damping="0.01" />
     </joint>
@@ -183,5 +183,5 @@
         <origin xyz="0 0 ${hand_length}" rpy="0 0 0" />
         <axis xyz="0 -1 0" />
-        <limit lower="${-2*PI/3}" upper="${2*PI/3}" effort="10" velocity="5.0" />
+        <limit lower="${-2*pi/3}" upper="${2*pi/3}" effort="10" velocity="5.0" />
         <dynamics friction="0.01" damping="0.01" />
     </joint>
@@ -191,5 +191,5 @@
         <origin xyz="0 0 ${hand_length}" rpy="0 0 0" />
         <axis xyz="0 -1 0" />
-        <limit lower="${-2*PI/3}" upper="${2*PI/3}" effort="10" velocity="5.0" />
+        <limit lower="${-2*pi/3}" upper="${2*pi/3}" effort="10" velocity="5.0" />
         <dynamics friction="0.01" damping="0.01" />
     </joint>
@@ -199,5 +199,5 @@
         <origin xyz="0 0 ${hand_length}" rpy="0 0 0" />
         <axis xyz="0 0 1" />
-        <limit lower="${-2*PI/3}" upper="${2*PI/3}" effort="10" velocity="5.0" />
+        <limit lower="${-2*pi/3}" upper="${2*pi/3}" effort="10" velocity="5.0" />
         <dynamics friction="0.01" damping="0.01" />
     </joint>
@@ -207,5 +207,5 @@
         <origin xyz="0 0.05 ${hand_length/8}"/>
         <axis xyz="1 0 0"/>
-        <limit lower="-${PI / 2}" upper="${PI / 2}"
+        <limit lower="-${pi / 2}" upper="${pi / 2}"
                effort="50" velocity="5.0"/>
     </joint>
@@ -215,5 +215,5 @@
         <origin xyz="0 -.05 ${hand_length/8}"/>
         <axis xyz="1 0 0"/>
-        <limit lower="-${PI / 2}" upper="${PI / 2}"
+        <limit lower="-${pi / 2}" upper="${pi / 2}"
                effort="50" velocity="5.0"/>
         <mimic joint="joint_4" multiplier="-1"/>

File: src/articubot_one/description/camera.xacro (robot description, xacro)
@@ -24,5 +24,5 @@
         <parent link="camera_link"/>
         <child link="camera_link_optical"/>
-        <origin xyz="0 0 0" rpy="${-PI/2} 0 ${-PI/2}"/>
+        <origin xyz="0 0 0" rpy="${-pi/2} 0 ${-pi/2}"/>
     </joint>
     <link name="camera_link_optical"></link>

File: src/articubot_one/description/depth_camera.xacro (robot description, xacro)
@@ -23,5 +23,5 @@
         <parent link="camera_link"/>
         <child link="camera_link_optical"/>
-        <origin xyz="0 0 0" rpy="${-PI/2} 0 ${-PI/2}"/>
+        <origin xyz="0 0 0" rpy="${-pi/2} 0 ${-pi/2}"/>
     </joint>
     <link name="camera_link_optical"></link>

File: src/articubot_one/description/face.xacro (robot description, xacro)
@@ -8,5 +8,5 @@
     <link name="face_link">
         <visual>
-            <origin xyz="0 0.05 0.01" rpy="0 ${PI/2} 0"/>
+            <origin xyz="0 0.05 0.01" rpy="0 ${pi/2} 0"/>
             <geometry>
                 <cylinder radius="0.01" length="0.002"/>
@@ -15,5 +15,5 @@
         </visual>
         <visual>
-            <origin xyz="0 -0.05 0.01" rpy="0 ${PI/2} 0"/>
+            <origin xyz="0 -0.05 0.01" rpy="0 ${pi/2} 0"/>
             <geometry>
                 <cylinder radius="0.01" length="0.002"/>

File: src/articubot_one/description/robot_core.xacro (robot description, xacro)
@@ -73,5 +73,5 @@
         <parent link="base_link"/>
         <child link="left_wheel"/>
-        <origin xyz="0 ${wheel_offset_y} 0" rpy="-${PI/2} 0 0" />
+        <origin xyz="0 ${wheel_offset_y} 0" rpy="-${pi/2} 0 0" />
         <axis xyz="0 0 1"/>
     </joint>
@@ -99,5 +99,5 @@
         <parent link="base_link"/>
         <child link="right_wheel"/>
-        <origin xyz="0 ${-wheel_offset_y} 0" rpy="${PI/2} 0 0" />
+        <origin xyz="0 ${-wheel_offset_y} 0" rpy="${pi/2} 0 0" />
         <axis xyz="0 0 -1"/>
     </joint>

File: src/articubot_one/description/ros2_control.xacro (robot description, xacro)
@@ -1,5 +1,5 @@
 <?xml version="1.0"?>
 <robot xmlns:xacro="http://www.ros.org/wiki/xacro">
-    <xacro:property name="PI" value="3.14159265359" />
+    <xacro:property name="pi" value="3.14159265359" />
     <xacro:unless value="$(arg sim_mode)">
         <ros2_control name="articubot" type="system">
@@ -35,6 +35,6 @@
             <joint name="arm_base_forearm_joint">
                 <command_interface name="position">
-                <param name="min">-${2*PI/3}</param>
-                <param name="max">${2*PI/3}</param>
+                <param name="min">-${2*pi/3}</param>
+                <param name="max">${2*pi/3}</param>
                 </command_interface>
                 <state_interface name="position"/>
@@ -42,6 +42,6 @@
             <joint name="forearm_hand_1_joint">
                 <command_interface name="position">
-                <param name="min">-${2*PI/3}</param>
-                <param name="max">${2*PI/3}</param>
+                <param name="min">-${2*pi/3}</param>
+                <param name="max">${2*pi/3}</param>
                 </command_interface>
                 <state_interface name="position"/>
@@ -49,6 +49,6 @@
             <joint name="forearm_hand_2_joint">
                 <command_interface name="position">
-                <param name="min">-${2*PI/3}</param>
-                <param name="max">${2*PI/3}</param>
+                <param name="min">-${2*pi/3}</param>
+                <param name="max">${2*pi/3}</param>
                 </command_interface>
                 <state_interface name="position"/>
@@ -56,6 +56,6 @@
             <joint name="forearm_hand_3_joint">
                 <command_interface name="position">
-                <param name="min">-${2*PI/3}</param>
-                <param name="max">${2*PI/3}</param>
+                <param name="min">-${2*pi/3}</param>
+                <param name="max">${2*pi/3}</param>
                 </command_interface>
                 <state_interface name="position"/>
@@ -63,6 +63,6 @@
              <joint name="forearm_claw_joint">
                 <command_interface name="position">
-                <param name="min">-${2*PI/3}</param>
-                <param name="max">${2*PI/3}</param>
+                <param name="min">-${2*pi/3}</param>
+                <param name="max">${2*pi/3}</param>
                 </command_interface>
                 <state_interface name="position"/>
@@ -70,6 +70,6 @@
             <joint name="joint_4">
                 <command_interface name="position">
-                <param name="min">-${PI / 2}</param>
-                <param name="max">${PI / 2}</param>
+                <param name="min">-${pi / 2}</param>
+                <param name="max">${pi / 2}</param>
                 </command_interface>
                 <state_interface name="position"/>
@@ -80,5 +80,5 @@
                 <command_interface name="position">
                 <param name="min">0.0</param>
-                <param name="max">${PI / 2}</param>
+                <param name="max">${pi / 2}</param>
                 </command_interface>
             </joint> -->
@@ -108,6 +108,6 @@
             <joint name="arm_base_forearm_joint">
                 <command_interface name="position">
-                <param name="min">-${PI / 2}</param>
-                <param name="max">${PI / 2}</param>
+                <param name="min">-${pi / 2}</param>
+                <param name="max">${pi / 2}</param>
                 </command_interface>
                 <state_interface name="position"/>
@@ -117,6 +117,6 @@
             <joint name="forearm_hand_1_joint">
                 <command_interface name="position">
-                <param name="min">-${PI / 2}</param>
-                <param name="max">${PI / 2}</param>
+                <param name="min">-${pi / 2}</param>
+                <param name="max">${pi / 2}</param>
                 </command_interface>
                 <state_interface name="position"/>
@@ -126,6 +126,6 @@
             <joint name="forearm_hand_2_joint">
                 <command_interface name="position">
-                <param name="min">-${PI / 2}</param>
-                <param name="max">${PI / 2}</param>
+                <param name="min">-${pi / 2}</param>
+                <param name="max">${pi / 2}</param>
                 </command_interface>
                 <state_interface name="position"/>
@@ -135,6 +135,6 @@
             <joint name="forearm_hand_3_joint">
                 <command_interface name="position">
-                <param name="min">-${PI / 2}</param>
-                <param name="max">${PI / 2}</param>
+                <param name="min">-${pi / 2}</param>
+                <param name="max">${pi / 2}</param>
                 </command_interface>
                 <state_interface name="position"/>
@@ -144,6 +144,6 @@
              <joint name="forearm_claw_joint">
                 <command_interface name="position">
-                <param name="min">-${PI / 2}</param>
-                <param name="max">${PI / 2}</param>
+                <param name="min">-${pi / 2}</param>
+                <param name="max">${pi / 2}</param>
                 </command_interface>
                 <state_interface name="position"/>
@@ -153,5 +153,5 @@
             <joint name="joint_4">
                 <command_interface name="position">
-                <param name="min">-${PI / 2}</param>
+                <param name="min">-${pi / 2}</param>
                 <param name="max">0.0</param>
                 </command_interface>
@@ -165,5 +165,5 @@
                 <command_interface name="position">
                 <param name="min">0.0</param>
-                <param name="max">${PI / 2}</param>
+                <param name="max">${pi / 2}</param>
                 </command_interface>
                 <state_interface name="position"/>

Commit message: 323

File: src/articubot_one/description/arm_robot.xacro (robot description, xacro)
@@ -167,5 +167,5 @@
         <origin xyz="0 0 ${arm_base_height}" rpy="0 0 0" />
         <axis xyz="0 0 1" />
-        <limit lower="${-2*pi/3}" upper="${2*pi/3}" effort="10" velocity="5.0" />
+        <limit lower="${-pi/2}" upper="${pi/2}" effort="10" velocity="5.0" />
         <dynamics friction="0.01" damping="0.01" />
     </joint>
@@ -175,5 +175,5 @@
         <origin xyz="0 0 ${forearm_length}" rpy="0 0 0" />
         <axis xyz="0 1 0" />
-        <limit lower="${-2*pi/3}" upper="${2*pi/3}" effort="10" velocity="5.0" />
+        <limit lower="${-pi/2}" upper="${pi/2}" effort="10" velocity="5.0" />
         <dynamics friction="0.01" damping="0.01" />
     </joint>
@@ -183,5 +183,5 @@
         <origin xyz="0 0 ${hand_length}" rpy="0 0 0" />
         <axis xyz="0 -1 0" />
-        <limit lower="${-2*pi/3}" upper="${2*pi/3}" effort="10" velocity="5.0" />
+        <limit lower="${-pi/2}" upper="${pi/2}" effort="10" velocity="5.0" />
         <dynamics friction="0.01" damping="0.01" />
     </joint>
@@ -191,5 +191,5 @@
         <origin xyz="0 0 ${hand_length}" rpy="0 0 0" />
         <axis xyz="0 -1 0" />
-        <limit lower="${-2*pi/3}" upper="${2*pi/3}" effort="10" velocity="5.0" />
+        <limit lower="${-pi/2}" upper="${pi/2}" effort="10" velocity="5.0" />
         <dynamics friction="0.01" damping="0.01" />
     </joint>
@@ -199,5 +199,5 @@
         <origin xyz="0 0 ${hand_length}" rpy="0 0 0" />
         <axis xyz="0 0 1" />
-        <limit lower="${-2*pi/3}" upper="${2*pi/3}" effort="10" velocity="5.0" />
+        <limit lower="${-pi/2}" upper="${pi/2}" effort="10" velocity="5.0" />
         <dynamics friction="0.01" damping="0.01" />
     </joint>
@@ -207,5 +207,5 @@
         <origin xyz="0 0.05 ${hand_length/8}"/>
         <axis xyz="1 0 0"/>
-        <limit lower="-${pi / 2}" upper="${pi / 2}"
+        <limit lower="-${PI / 2}" upper="${PI / 2}"
                effort="50" velocity="5.0"/>
     </joint>
@@ -215,5 +215,5 @@
         <origin xyz="0 -.05 ${hand_length/8}"/>
         <axis xyz="1 0 0"/>
-        <limit lower="-${pi / 2}" upper="${pi / 2}"
+        <limit lower="-${PI / 2}" upper="${PI / 2}"
                effort="50" velocity="5.0"/>
         <mimic joint="joint_4" multiplier="-1"/>

Commit message: we

File: src/articubot_one/description/arm_robot.xacro (robot description, xacro)
@@ -18,5 +18,5 @@
         </inertial>
     </xacro:macro>
-    <xacro:property name="pi" value="3.14159265359" />
+    <xacro:property name="PI" value="3.14159265359" />
     <xacro:property name="effort" value="30.0" />
     <xacro:property name="velocity" value="10.0" />
@@ -167,5 +167,5 @@
         <origin xyz="0 0 ${arm_base_height}" rpy="0 0 0" />
         <axis xyz="0 0 1" />
-        <limit lower="${-pi/2}" upper="${pi/2}" effort="10" velocity="5.0" />
+        <limit lower="${-PI/2}" upper="${PI/2}" effort="10" velocity="5.0" />
         <dynamics friction="0.01" damping="0.01" />
     </joint>
@@ -175,5 +175,5 @@
         <origin xyz="0 0 ${forearm_length}" rpy="0 0 0" />
         <axis xyz="0 1 0" />
-        <limit lower="${-pi/2}" upper="${pi/2}" effort="10" velocity="5.0" />
+        <limit lower="${-PI/2}" upper="${PI/2}" effort="10" velocity="5.0" />
         <dynamics friction="0.01" damping="0.01" />
     </joint>
@@ -183,5 +183,5 @@
         <origin xyz="0 0 ${hand_length}" rpy="0 0 0" />
         <axis xyz="0 -1 0" />
-        <limit lower="${-pi/2}" upper="${pi/2}" effort="10" velocity="5.0" />
+        <limit lower="${-PI/2}" upper="${PI/2}" effort="10" velocity="5.0" />
         <dynamics friction="0.01" damping="0.01" />
     </joint>
@@ -191,5 +191,5 @@
         <origin xyz="0 0 ${hand_length}" rpy="0 0 0" />
         <axis xyz="0 -1 0" />
-        <limit lower="${-pi/2}" upper="${pi/2}" effort="10" velocity="5.0" />
+        <limit lower="${-PI/2}" upper="${PI/2}" effort="10" velocity="5.0" />
         <dynamics friction="0.01" damping="0.01" />
     </joint>
@@ -199,5 +199,5 @@
         <origin xyz="0 0 ${hand_length}" rpy="0 0 0" />
         <axis xyz="0 0 1" />
-        <limit lower="${-pi/2}" upper="${pi/2}" effort="10" velocity="5.0" />
+        <limit lower="${-PI/2}" upper="${PI/2}" effort="10" velocity="5.0" />
         <dynamics friction="0.01" damping="0.01" />
     </joint>
