Commit message: 33

File: src/articubot_one/description/arm_robot.xacro (robot description, xacro)
@@ -18,5 +18,4 @@
         </inertial>
     </xacro:macro>
-    <xacro:property name="PI" value="3.14159265359" />
     <xacro:property name="effort" value="30.0" />
     <xacro:property name="velocity" value="10.0" />
@@ -167,5 +166,5 @@
         <origin xyz="0 0 ${arm_base_height}" rpy="0 0 0" />
         <axis xyz="0 0 1" />
-        <limit lower="${-PI/2}" upper="${PI/2}" effort="10" velocity="5.0" />
+        <limit lower="${-pi/2}" upper="${pi/2}" effort="10" velocity="5.0" />
         <dynamics friction="0.01" damping="0.01" />
     </joint>
@@ -175,5 +174,5 @@
         <origin xyz="0 0 ${forearm_length}" rpy="0 0 0" />
         <axis xyz="0 1 0" />
-        <limit lower="${-PI/2}" upper="${PI/2}" effort="10" velocity="5.0" />
+        <limit lower="${-pi/2}" upper="${pi/2}" effort="10" velocity="5.0" />
         <dynamics friction="0.01" damping="0.01" />
     </joint>
@@ -183,5 +182,5 @@
         <origin xyz="0 0 ${hand_length}" rpy="0 0 0" />
         <axis xyz="0 -1 0" />
-        <limit lower="${-PI/2}" upper="${PI/2}" effort="10" velocity="5.0" />
+        <limit lower="${-pi/2}" upper="${pi/2}" effort="10" velocity="5.0" />
         <dynamics friction="0.01" damping="0.01" />
     </joint>
@@ -191,5 +190,5 @@
         <origin xyz="0 0 ${hand_length}" rpy="0 0 0" />
         <axis xyz="0 -1 0" />
-        <limit lower="${-PI/2}" upper="${PI/2}" effort="10" velocity="5.0" />
+        <limit lower="${-pi/2}" upper="${pi/2}" effort="10" velocity="5.0" />
         <dynamics friction="0.01" damping="0.01" />
     </joint>
@@ -199,5 +198,5 @@
         <origin xyz="0 0 ${hand_length}" rpy="0 0 0" />
         <axis xyz="0 0 1" />
-        <limit lower="${-PI/2}" upper="${PI/2}" effort="10" velocity="5.0" />
+        <limit lower="${-pi/2}" upper="${pi/2}" effort="10" velocity="5.0" />
         <dynamics friction="0.01" damping="0.01" />
     </joint>
@@ -207,5 +206,5 @@
         <origin xyz="0 0.05 ${hand_length/8}"/>
         <axis xyz="1 0 0"/>
-        <limit lower="-${PI / 2}" upper="${PI / 2}"
+        <limit lower="-${pi / 2}" upper="${pi / 2}"
                effort="50" velocity="5.0"/>
     </joint>
@@ -215,5 +214,5 @@
         <origin xyz="0 -.05 ${hand_length/8}"/>
         <axis xyz="1 0 0"/>
-        <limit lower="-${PI / 2}" upper="${PI / 2}"
+        <limit lower="-${pi / 2}" upper="${pi / 2}"
                effort="50" velocity="5.0"/>
         <mimic joint="joint_4" multiplier="-1"/>

File: src/articubot_one/description/ros2_control.xacro (robot description, xacro)
@@ -1,5 +1,4 @@
 <?xml version="1.0"?>
 <robot xmlns:xacro="http://www.ros.org/wiki/xacro">
-    <xacro:property name="PI" value="3.14159265359" />
     <xacro:unless value="$(arg sim_mode)">
         <ros2_control name="articubot" type="system">
@@ -35,6 +34,6 @@
             <joint name="arm_base_forearm_joint">
                 <command_interface name="position">
-                <param name="min">-${2*PI/3}</param>
-                <param name="max">${2*PI/3}</param>
+                <param name="min">-${2*pi/3}</param>
+                <param name="max">${2*pi/3}</param>
                 </command_interface>
                 <state_interface name="position"/>
@@ -42,6 +41,6 @@
             <joint name="forearm_hand_1_joint">
                 <command_interface name="position">
-                <param name="min">-${2*PI/3}</param>
-                <param name="max">${2*PI/3}</param>
+                <param name="min">-${2*pi/3}</param>
+                <param name="max">${2*pi/3}</param>
                 </command_interface>
                 <state_interface name="position"/>
@@ -49,6 +48,6 @@
             <joint name="forearm_hand_2_joint">
                 <command_interface name="position">
-                <param name="min">-${2*PI/3}</param>
-                <param name="max">${2*PI/3}</param>
+                <param name="min">-${2*pi/3}</param>
+                <param name="max">${2*pi/3}</param>
                 </command_interface>
                 <state_interface name="position"/>
@@ -56,6 +55,6 @@
             <joint name="forearm_hand_3_joint">
                 <command_interface name="position">
-                <param name="min">-${2*PI/3}</param>
-                <param name="max">${2*PI/3}</param>
+                <param name="min">-${2*pi/3}</param>
+                <param name="max">${2*pi/3}</param>
                 </command_interface>
                 <state_interface name="position"/>
@@ -63,6 +62,6 @@
              <joint name="forearm_claw_joint">
                 <command_interface name="position">
-                <param name="min">-${2*PI/3}</param>
-                <param name="max">${2*PI/3}</param>
+                <param name="min">-${2*pi/3}</param>
+                <param name="max">${2*pi/3}</param>
                 </command_interface>
                 <state_interface name="position"/>
@@ -70,6 +69,6 @@
             <joint name="joint_4">
                 <command_interface name="position">
-                <param name="min">-${PI / 2}</param>
-                <param name="max">${PI / 2}</param>
+                <param name="min">-${pi / 2}</param>
+                <param name="max">${pi / 2}</param>
                 </command_interface>
                 <state_interface name="position"/>
@@ -80,5 +79,5 @@
                 <command_interface name="position">
                 <param name="min">0.0</param>
-                <param name="max">${PI / 2}</param>
+                <param name="max">${pi / 2}</param>
                 </command_interface>
             </joint> -->
@@ -108,6 +107,6 @@
             <joint name="arm_base_forearm_joint">
                 <command_interface name="position">
-                <param name="min">-${PI / 2}</param>
-                <param name="max">${PI / 2}</param>
+                <param name="min">-${pi / 2}</param>
+                <param name="max">${pi / 2}</param>
                 </command_interface>
                 <state_interface name="position"/>
@@ -117,6 +116,6 @@
             <joint name="forearm_hand_1_joint">
                 <command_interface name="position">
-                <param name="min">-${PI / 2}</param>
-                <param name="max">${PI / 2}</param>
+                <param name="min">-${pi / 2}</param>
+                <param name="max">${pi / 2}</param>
                 </command_interface>
                 <state_interface name="position"/>
@@ -126,6 +125,6 @@
             <joint name="forearm_hand_2_joint">
                 <command_interface name="position">
-                <param name="min">-${PI / 2}</param>
-                <param name="max">${PI / 2}</param>
+                <param name="min">-${pi / 2}</param>
+                <param name="max">${pi / 2}</param>
                 </command_interface>
                 <state_interface name="position"/>
@@ -135,6 +134,6 @@
             <joint name="forearm_hand_3_joint">
                 <command_interface name="position">
-                <param name="min">-${PI / 2}</param>
-                <param name="max">${PI / 2}</param>
+                <param name="min">-${pi / 2}</param>
+                <param name="max">${pi / 2}</param>
                 </command_interface>
                 <state_interface name="position"/>
@@ -144,6 +143,6 @@
              <joint name="forearm_claw_joint">
                 <command_interface name="position">
-                <param name="min">-${PI / 2}</param>
-                <param name="max">${PI / 2}</param>
+                <param name="min">-${pi / 2}</param>
+                <param name="max">${pi / 2}</param>
                 </command_interface>
                 <state_interface name="position"/>
@@ -153,5 +152,5 @@
             <joint name="joint_4">
                 <command_interface name="position">
-                <param name="min">-${PI / 2}</param>
+                <param name="min">-${pi / 2}</param>
                 <param name="max">0.0</param>
                 </command_interface>
@@ -165,5 +164,5 @@
                 <command_interface name="position">
                 <param name="min">0.0</param>
-                <param name="max">${PI / 2}</param>
+                <param name="max">${pi / 2}</param>
                 </command_interface>
                 <state_interface name="position"/>

Commit message: 332

File: src/articubot_one/description/arm_robot.xacro (robot description, xacro)
@@ -166,5 +166,5 @@
         <origin xyz="0 0 ${arm_base_height}" rpy="0 0 0" />
         <axis xyz="0 0 1" />
-        <limit lower="${-pi/2}" upper="${pi/2}" effort="10" velocity="5.0" />
+        <limit lower="${-2*pi/3}" upper="${2*pi/3}" effort="10" velocity="5.0" />
         <dynamics friction="0.01" damping="0.01" />
     </joint>
@@ -174,5 +174,5 @@
         <origin xyz="0 0 ${forearm_length}" rpy="0 0 0" />
         <axis xyz="0 1 0" />
-        <limit lower="${-pi/2}" upper="${pi/2}" effort="10" velocity="5.0" />
+        <limit lower="${-2*pi/3}" upper="${2*pi/3}" effort="10" velocity="5.0" />
         <dynamics friction="0.01" damping="0.01" />
     </joint>
@@ -182,5 +182,5 @@
         <origin xyz="0 0 ${hand_length}" rpy="0 0 0" />
         <axis xyz="0 -1 0" />
-        <limit lower="${-pi/2}" upper="${pi/2}" effort="10" velocity="5.0" />
+        <limit lower="${-2*pi/3}" upper="${2*pi/3}" effort="10" velocity="5.0" />
         <dynamics friction="0.01" damping="0.01" />
     </joint>
@@ -190,5 +190,5 @@
         <origin xyz="0 0 ${hand_length}" rpy="0 0 0" />
         <axis xyz="0 -1 0" />
-        <limit lower="${-pi/2}" upper="${pi/2}" effort="10" velocity="5.0" />
+        <limit lower="${-2*pi/3}" upper="${2*pi/3}" effort="10" velocity="5.0" />
         <dynamics friction="0.01" damping="0.01" />
     </joint>
@@ -198,5 +198,5 @@
         <origin xyz="0 0 ${hand_length}" rpy="0 0 0" />
         <axis xyz="0 0 1" />
-        <limit lower="${-pi/2}" upper="${pi/2}" effort="10" velocity="5.0" />
+        <limit lower="${-2*pi/3}" upper="${2*pi/3}" effort="10" velocity="5.0" />
         <dynamics friction="0.01" damping="0.01" />
     </joint>

Commit message: 32

File: src/articubot_one/description/arm_robot.xacro (robot description, xacro)
@@ -201,20 +201,20 @@
         <dynamics friction="0.01" damping="0.01" />
     </joint>
-    <joint name ="joint_4" type="revolute">
+    <joint name="joint_4" type="revolute">
         <parent link="claw_support"/>
-        <child link = "gripper_right"/>
-        <origin xyz="0 0.05 ${hand_length/8}"/>
+        <child link="gripper_right"/>
+        <origin xyz="0 0.05 ${hand_length/8}" rpy="0 0 0"/>
         <axis xyz="1 0 0"/>
-        <limit lower="-${pi / 2}" upper="${pi / 2}"
-               effort="50" velocity="5.0"/>
-    </joint>
-    <joint name ="joint_5" type="revolute">
+        <limit lower="-${pi/2}" upper="${pi/2}" effort="10" velocity="5.0"/>
+        <dynamics friction="0.01" damping="0.01" />
+    </joint>
+    <joint name="joint_5" type="revolute">
         <parent link="claw_support"/>
-        <child link = "gripper_left"/>
-        <origin xyz="0 -.05 ${hand_length/8}"/>
+        <child link="gripper_left"/>
+        <origin xyz="0 -0.05 ${hand_length/8}" rpy="0 0 0"/>
         <axis xyz="1 0 0"/>
-        <limit lower="-${pi / 2}" upper="${pi / 2}"
-               effort="50" velocity="5.0"/>
+        <limit lower="-${pi/2}" upper="${pi/2}" effort="10" velocity="5.0"/>
         <mimic joint="joint_4" multiplier="-1"/>
+        <dynamics friction="0.01" damping="0.01" />
     </joint>
     <gazebo reference="arm_base_link">

Commit message: 323

File: src/articubot_one/description/arm_robot.xacro (robot description, xacro)
@@ -166,5 +166,5 @@
         <origin xyz="0 0 ${arm_base_height}" rpy="0 0 0" />
         <axis xyz="0 0 1" />
-        <limit lower="${-2*pi/3}" upper="${2*pi/3}" effort="10" velocity="5.0" />
+        <limit lower="${-pi}" upper="${pi}" effort="10" velocity="5.0" />
         <dynamics friction="0.01" damping="0.01" />
     </joint>
@@ -174,5 +174,5 @@
         <origin xyz="0 0 ${forearm_length}" rpy="0 0 0" />
         <axis xyz="0 1 0" />
-        <limit lower="${-2*pi/3}" upper="${2*pi/3}" effort="10" velocity="5.0" />
+        <limit lower="${-pi}" upper="${pi}" effort="10" velocity="5.0" />
         <dynamics friction="0.01" damping="0.01" />
     </joint>
@@ -182,5 +182,5 @@
         <origin xyz="0 0 ${hand_length}" rpy="0 0 0" />
         <axis xyz="0 -1 0" />
-        <limit lower="${-2*pi/3}" upper="${2*pi/3}" effort="10" velocity="5.0" />
+        <limit lower="${-pi}" upper="${pi}" effort="10" velocity="5.0" />
         <dynamics friction="0.01" damping="0.01" />
     </joint>
@@ -190,5 +190,5 @@
         <origin xyz="0 0 ${hand_length}" rpy="0 0 0" />
         <axis xyz="0 -1 0" />
-        <limit lower="${-2*pi/3}" upper="${2*pi/3}" effort="10" velocity="5.0" />
+        <limit lower="${-pi}" upper="${pi}" effort="10" velocity="5.0" />
         <dynamics friction="0.01" damping="0.01" />
     </joint>
@@ -198,5 +198,5 @@
         <origin xyz="0 0 ${hand_length}" rpy="0 0 0" />
         <axis xyz="0 0 1" />
-        <limit lower="${-2*pi/3}" upper="${2*pi/3}" effort="10" velocity="5.0" />
+        <limit lower="${-pi}" upper="${pi}" effort="10" velocity="5.0" />
         <dynamics friction="0.01" damping="0.01" />
     </joint>

Commit message: 232

File: src/articubot_one/description/arm_robot.xacro (robot description, xacro)
@@ -166,5 +166,5 @@
         <origin xyz="0 0 ${arm_base_height}" rpy="0 0 0" />
         <axis xyz="0 0 1" />
-        <limit lower="${-pi}" upper="${pi}" effort="10" velocity="5.0" />
+        <limit lower="${-2*pi/3}" upper="${2*pi/3}" effort="10" velocity="5.0" />
         <dynamics friction="0.01" damping="0.01" />
     </joint>
@@ -174,5 +174,5 @@
         <origin xyz="0 0 ${forearm_length}" rpy="0 0 0" />
         <axis xyz="0 1 0" />
-        <limit lower="${-pi}" upper="${pi}" effort="10" velocity="5.0" />
+        <limit lower="${-2*pi/3}" upper="${2*pi/3}" effort="10" velocity="5.0" />
         <dynamics friction="0.01" damping="0.01" />
     </joint>
@@ -182,5 +182,5 @@
         <origin xyz="0 0 ${hand_length}" rpy="0 0 0" />
         <axis xyz="0 -1 0" />
-        <limit lower="${-pi}" upper="${pi}" effort="10" velocity="5.0" />
+        <limit lower="${-2*pi/3}" upper="${2*pi/3}" effort="10" velocity="5.0" />
         <dynamics friction="0.01" damping="0.01" />
     </joint>
@@ -190,5 +190,5 @@
         <origin xyz="0 0 ${hand_length}" rpy="0 0 0" />
         <axis xyz="0 -1 0" />
-        <limit lower="${-pi}" upper="${pi}" effort="10" velocity="5.0" />
+        <limit lower="${-2*pi/3}" upper="${2*pi/3}" effort="10" velocity="5.0" />
         <dynamics friction="0.01" damping="0.01" />
     </joint>
@@ -198,5 +198,5 @@
         <origin xyz="0 0 ${hand_length}" rpy="0 0 0" />
         <axis xyz="0 0 1" />
-        <limit lower="${-pi}" upper="${pi}" effort="10" velocity="5.0" />
+        <limit lower="${-2*pi/3}" upper="${2*pi/3}" effort="10" velocity="5.0" />
         <dynamics friction="0.01" damping="0.01" />
     </joint>
@@ -206,5 +206,5 @@
         <origin xyz="0 0.05 ${hand_length/8}" rpy="0 0 0"/>
         <axis xyz="1 0 0"/>
-        <limit lower="-${pi/2}" upper="${pi/2}" effort="10" velocity="5.0"/>
+        <limit lower="-${2*pi/3/2}" upper="${2*pi/3/2}" effort="10" velocity="5.0"/>
         <dynamics friction="0.01" damping="0.01" />
     </joint>
@@ -214,5 +214,5 @@
         <origin xyz="0 -0.05 ${hand_length/8}" rpy="0 0 0"/>
         <axis xyz="1 0 0"/>
-        <limit lower="-${pi/2}" upper="${pi/2}" effort="10" velocity="5.0"/>
+        <limit lower="-${2*pi/3/2}" upper="${2*pi/3/2}" effort="10" velocity="5.0"/>
         <mimic joint="joint_4" multiplier="-1"/>
         <dynamics friction="0.01" damping="0.01" />
